Commit message: spheres configuration, with collision checking and visualization of collision forces.

File: model/bifrank_robot.urdf (robot description, URDF)
Before this commit: robot bifrank_robot, 22 links, 21 joints
Links:
- link lewis_fr3_link0: geometry collision sphere radius=0.09; visual mesh filename=package://model/meshes/visual/link0.dae
- link lewis_fr3_link1: geometry collision sphere radius=0.07; collision sphere radius=0.07
- link lewis_fr3_link2: geometry collision sphere radius=0.07; visual mesh filename=package://model/meshes/visual/link2.dae
- link lewis_fr3_link3: geometry collision sphere radius=0.06; collision sphere radius=0.06
- link lewis_fr3_link4: geometry collision sphere radius=0.06; collision sphere radius=0.06
- link lewis_fr3_link5: geometry collision sphere radius=0.06; collision sphere radius=0.06
- link lewis_fr3_link6: geometry collision sphere radius=0.05; visual mesh filename=package://model/meshes/visual/link6.dae
- link lewis_fr3_link7: geometry collision sphere radius=0.04; visual mesh filename=package://model/meshes/visual/link7.dae
- link richard_fr3_link0: geometry collision sphere radius=0.09; visual mesh filename=package://model/meshes/visual/link0.dae
- link richard_fr3_link1: geometry collision sphere radius=0.07; collision sphere radius=0.07
- link richard_fr3_link2: geometry collision sphere radius=0.07; visual mesh filename=package://model/meshes/visual/link2.dae
- link richard_fr3_link3: geometry collision sphere radius=0.06; collision sphere radius=0.06
- link richard_fr3_link4: geometry collision sphere radius=0.06; collision sphere radius=0.06
- link richard_fr3_link5: geometry collision sphere radius=0.06; collision sphere radius=0.06
- link richard_fr3_link6: geometry collision sphere radius=0.05; visual mesh filename=package://model/meshes/visual/link6.dae
- link richard_fr3_link7: geometry collision sphere radius=0.04; visual mesh filename=package://model/meshes/visual/link7.dae
