Commit message: foam spheres

File: model/bifrank_clean.urdf (robot description, URDF)
Before this commit: robot bifrank_robot, 22 links, 21 joints
Links:
- link base_link: geometry collision box size=0.5 0.5 0.1; visual box size=0.5 0.5 0.1
- link lewis_fr3_link0: geometry collision mesh filename=package://model/meshes/collision/link0.stl; visual mesh filename=package://model/meshes/visual/link0.dae
- link lewis_fr3_link1: geometry collision mesh filename=package://model/meshes/collision/link1.stl; visual mesh filename=package://model/meshes/visual/link1.dae
- link lewis_fr3_link2: geometry collision mesh filename=package://model/meshes/collision/link2.stl; visual mesh filename=package://model/meshes/visual/link2.dae
- link lewis_fr3_link3: geometry collision mesh filename=package://model/meshes/collision/link3.stl; visual mesh filename=package://model/meshes/visual/link3.dae
- link lewis_fr3_link4: geometry collision mesh filename=package://model/meshes/collision/link4.stl; visual mesh filename=package://model/meshes/visual/link4.dae
- link lewis_fr3_link5: geometry collision mesh filename=package://model/meshes/collision/link5.stl; visual mesh filename=package://model/meshes/visual/link5.dae
- link lewis_fr3_link6: geometry collision mesh filename=package://model/meshes/collision/link6.stl; visual mesh filename=package://model/meshes/visual/link6.dae
- link lewis_fr3_link7: geometry collision mesh filename=package://model/meshes/collision/link7.stl; visual mesh filename=package://model/meshes/visual/link7.dae
- link richard_fr3_link0: geometry collision mesh filename=package://model/meshes/collision/link0.stl; visual mesh filename=package://model/meshes/visual/link0.dae
- link richard_fr3_link1: geometry collision mesh filename=package://model/meshes/collision/link1.stl; visual mesh filename=package://model/meshes/visual/link1.dae
- link richard_fr3_link2: geometry collision mesh filename=package://model/meshes/collision/link2.stl; visual mesh filename=package://model/meshes/visual/link2.dae
- link richard_fr3_link3: geometry collision mesh filename=package://model/meshes/collision/link3.stl; visual mesh filename=package://model/meshes/visual/link3.dae
- link richard_fr3_link4: geometry collision mesh filename=package://model/meshes/collision/link4.stl; visual mesh filename=package://model/meshes/visual/link4.dae
- link richard_fr3_link5: geometry collision mesh filename=package://model/meshes/collision/link5.stl; visual mesh filename=package://model/meshes/visual/link5.dae
- link richard_fr3_link6: geometry collision mesh filename=package://model/meshes/collision/link6.stl; visual mesh filename=package://model/meshes/visual/link6.dae
- link richard_fr3_link7: geometry collision mesh filename=package://model/meshes/collision/link7.stl; visual mesh filename=package://model/meshes/visual/link7.dae
